File: LearningKiCAD.kicad_sch (KiCad schematic)
At the start: 4 parts, among them U1 ADA4075-2

Commit message: Autosave
Connections:
- net Vcc: now also U1.8 (V+)
Changed lines of the file:
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@@
+	(wire
+		(pts
+			(xy 44.45 38.1) (xy 44.45 48.26)
+		)
+		(stroke
+			(width 0)
+			(type default)
+		)
+	)
 	(wire
 		(pts
@@
 					(unit 1)
 				)
+			)
+		)
+	)
+	(symbol
+		(lib_id "power:VDC")
+		(at 44.45 72.39 0)
+		(mirror x)
+		(unit 1)
+		(body_style 1)
+		(exclude_from_sim no)
+		(in_bom yes)
+		(on_board yes)
+		(in_pos_files yes)
+		(dnp no)
+		(property "Reference" "#PWR06"
+			(at 44.45 68.58 0)
+			(hide yes)
+			(show_name no)
+			(do_not_autoplace no)
+			(effects
+				(font
+					(size 1.27 1.27)
+				)
+			)
+		)
+		(property "Value" "Vdd"
+			(at 44.45 77.47 0)
+			(show_name no)
+			(do_not_autoplace no)
+			(effects
+				(font
+					(size 1.27 1.27)
+				)
+			)
+		)
+		(property "Footprint" ""
+			(at 44.45 72.39 0)
+			(hide yes)
+			(show_name no)
+			(do_not_autoplace no)
+			(effects
+				(font
+					(size 1.27 1.27)
+				)
+			)
+		)
+		(property "Datasheet" ""
+			(at 44.45 72.39 0)
+			(hide yes)
+			(show_name no)
+			(do_not_autoplace no)
+			(effects
+				(font
+					(size 1.27 1.27)
+				)
+			)
+		)
+		(property "Description" "Power symbol creates a global label with name \"VDC\""
+			(at 44.45 72.39 0)
+			(hide yes)
+			(show_name no)
+			(do_not_autoplace no)
+			(effects
+				(font
+					(size 1.27 1.27)
+				)
+			)
+		)
+		(pin "1"
+		)
+		(instances
+			(project "LearningKiCAD"
+				(path "/61d3d1c1-c158-4903-81b9-c929de3a922a"
+					(reference "#PWR06")
+					(unit 1)
+				)

Commit message: Autosave
Connections:
- net Vdd: now also U1.4 (V-)
Changed lines of the file:
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@@
 	(wire
 		(pts
-			(xy 44.45 64.77) (xy 44.45 63.5)
+			(xy 144.78 78.74) (xy 146.05 78.74)
 		)
 		(stroke
@@
 	(wire
 		(pts
-			(xy 144.78 78.74) (xy 146.05 78.74)
+			(xy 44.45 63.5) (xy 44.45 72.39)
 		)
 		(stroke

Commit message: Autosave
Parts:
- V2: value 1 -> 15
Changed lines of the file:
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@@
 			)
 		)
-		(property "Value" "1"
+		(property "Value" "15"
 			(at 74.93 44.3201 0)
 			(show_name no)

Commit message: Autosave
Parts:
- V3: value 1 -> 15
Changed lines of the file:
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@@
 			)
 		)
-		(property "Value" "1"
+		(property "Value" "15"
 			(at 74.93 62.1001 0)
 			(show_name no)

Commit message: Close: 4 files changed LearningKiCAD.kicad_pcb 2/0/0 LearningKiCAD.kicad_prl 138/0/0 LearningKiCAD.kicad_pro 664/0/0 LearningKiCAD.kicad_sch 0/2205/3
Parts:
- removed U1: ADA4075-2, symbol Amplifier_Operational:ADA4075-2
- removed V1: VSIN, symbol Simulation_SPICE:VSIN
- removed V2, V3: 15, symbol Simulation_SPICE:VDC

Commit message: Add README.txt for KiCad Local History Directory
This file explains the purpose of the local history directory,
how to access previous versions of project files, and instructions
for disabling the automatic backup feature. It also notes that
the directory can be deleted if the history is no longer needed.
Parts:
- added U1: ADA4075-2, symbol Amplifier_Operational:ADA4075-2
- added V1: VSIN, symbol Simulation_SPICE:VSIN
- added V2, V3: 15, symbol Simulation_SPICE:VDC
Connections:
- new net: U1.3 (+), V1.1
- new net GND: V1.2, V2.2, V3.1
- new net Vcc: U1.8 (V+), V2.1
- new net Vdd: U1.4 (V-), V3.2
- new net out: U1.1, U1.2 (-)

Commit message: Autosave
Parts:
- removed U1: ADA4075-2, symbol Amplifier_Operational:ADA4075-2
- removed V1: VSIN, symbol Simulation_SPICE:VSIN
- removed V2, V3: 15, symbol Simulation_SPICE:VDC
- added U1: ${SIM.PARAMS}, symbol Simulation_SPICE:OPAMP
