File: LearningKiCAD.kicad_sch (KiCad schematic)
At the start: 4 parts, among them U1 ${SIM.PARAMS}

Commit message: Autosave
Parts:
- V2: value 1 -> 15
Changed lines of the file:
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@@
 			)
 		)
-		(property "Value" "1"
+		(property "Value" "15"
 			(at 35.56 63.3701 0)
 			(show_name no)

Commit message: Autosave
Parts:
- V3: value 1 -> 15
Changed lines of the file:
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@@
 			)
 		)
-		(property "Value" "1"
+		(property "Value" "15"
 			(at 35.56 90.0401 0)
 			(show_name no)

Commit message: Autosave
Connections:
- net GND: no longer U1.2 (-)
Changed lines of the file:
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@@
-	(wire
-		(pts
-			(xy 116.84 74.93) (xy 121.92 74.93)
-		)
-		(stroke
-			(width 0)
-			(type default)
-		)
-	)
 	(wire
 		(pts
@@
 		)
 		(stroke
-			(width 0)
-			(type default)
-		)
-	)
-	(wire
-		(pts
-			(xy 116.84 93.98) (xy 116.84 74.93)
-		)
-		(stroke

Commit message: SCH Save
Connections:
- net GND: now also U1.2 (-)
Changed lines of the file:
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@@
+	(wire
+		(pts
+			(xy 116.84 93.98) (xy 116.84 74.93)
+		)
+		(stroke
+			(width 0)
+			(type default)
+		)
+	)
 	(wire
 		(pts
@@
 		)
 		(stroke
+			(width 0)
+			(type default)
+		)
+	)
+	(wire
+		(pts
+			(xy 116.84 74.93) (xy 121.92 74.93)
+		)
+		(stroke

Commit message: Autosave
Connections:
- net GND: no longer U1.2 (-)
Changed lines of the file:
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@@
-	(wire
-		(pts
-			(xy 116.84 93.98) (xy 116.84 74.93)
-		)
-		(stroke
-			(width 0)
-			(type default)
-		)
-	)
 	(wire
 		(pts
 			(xy 31.75 93.98) (xy 31.75 124.46)
-		)
-		(stroke
-			(width 0)
-			(type default)
-		)
-	)
-	(wire
-		(pts
-			(xy 116.84 74.93) (xy 121.92 74.93)
 		)
 		(stroke
@@
 		)
 	)
-	(symbol
-		(lib_id "power:GND")
-		(at 116.84 93.98 0)
-		(unit 1)
-		(body_style 1)
-		(exclude_from_sim no)
-		(in_bom yes)
-		(on_board yes)
-		(in_pos_files yes)
-		(dnp no)
-		(fields_autoplaced yes)
-		(property "Reference" "#PWR03"
-			(at 116.84 100.33 0)
-			(hide yes)
-			(show_name no)
-			(do_not_autoplace no)
-			(effects
-				(font
-					(size 1.27 1.27)
-				)
-			)
-		)
-		(property "Value" "GND"
-			(at 116.84 99.06 0)
-			(show_name no)
-			(do_not_autoplace no)
-			(effects
-				(font
-					(size 1.27 1.27)
-				)
-			)
-		)
-		(property "Footprint" ""
-			(at 116.84 93.98 0)
-			(hide yes)
-			(show_name no)
-			(do_not_autoplace no)
-			(effects
-				(font
-					(size 1.27 1.27)
-				)
-			)
-		)
-		(property "Datasheet" ""
-			(at 116.84 93.98 0)
-			(hide yes)
-			(show_name no)
-			(do_not_autoplace no)
-			(effects
-				(font
-					(size 1.27 1.27)
-				)
-			)
-		)
-		(property "Description" "Power symbol creates a global label with name \"GND\" , ground"
-			(at 116.84 93.98 0)
-			(hide yes)
-			(show_name no)
-			(do_not_autoplace no)
-			(effects
-				(font
-					(size 1.27 1.27)
-				)
-			)
-		)
-		(pin "1"
-		)
-		(instances
-			(project "LearningKiCAD"
-				(path "/61d3d1c1-c158-4903-81b9-c929de3a922a"
-					(reference "#PWR03")
-					(unit 1)
-				)
-			)
-		)
-	)

Commit message: SCH Save
Connections:
- net GND: now also U1.2 (-)
Changed lines of the file:
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@@
+	)
+	(junction
+		(at 59.69 87.63)
+		(diameter 0)
+		(color 0 0 0 0)
 	)
 	(junction
@@
 	(wire
 		(pts
-			(xy 59.69 80.01) (xy 59.69 93.98)
+			(xy 59.69 87.63) (xy 59.69 93.98)
+		)
+		(stroke
+			(width 0)
+			(type default)
+		)
+	)
+	(wire
+		(pts
+			(xy 59.69 80.01) (xy 59.69 87.63)
 		)
 		(stroke
@@
 	(wire
 		(pts
+			(xy 121.92 74.93) (xy 121.92 87.63)
+		)
+		(stroke
+			(width 0)
+			(type default)
+		)
+	)
+	(wire
+		(pts
 			(xy 144.78 67.31) (xy 144.78 72.39)
 		)
@@
 		)
 		(stroke
+			(width 0)
+			(type default)
+		)
+	)
+	(wire
+		(pts
+			(xy 121.92 87.63) (xy 59.69 87.63)
+		)
+		(stroke

Commit message: Autosave
Connections:
- net cc: no longer U1.3 (V+), V2.1
Changed lines of the file:
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@@
 	(paper "A4")
-	(junction
-		(at 87.63 33.02)
-		(diameter 0)
-		(color 0 0 0 0)
-	)
 	(junction
 		(at 59.69 87.63)
@@
 		(pts
 			(xy 59.69 80.01) (xy 59.69 87.63)
-		)
-		(stroke
-			(width 0)
-			(type default)
-		)
-	)
-	(wire
-		(pts
-			(xy 87.63 33.02) (xy 127 33.02)
 		)
 		(stroke
@@
 		)
 		(stroke
-			(width 0)
-			(type default)
-		)
-	)
-	(wire
-		(pts
-			(xy 31.75 33.02) (xy 87.63 33.02)
-		)
-		(stroke
-			(width 0)
-			(type default)
-		)
-	)
-	(wire
-		(pts
-			(xy 127 33.02) (xy 127 64.77)
-		)
-		(stroke
